Commit message: Adding visualisation for end effector

File: src/linear_gripper_visualiser/urdf/ur_with_gripper.urdf.xacro (robot description, xacro)
@@ -1,6 +1,11 @@
-<?xml version="1.0"?>
-<robot name="gripper">
-  <!-- Base -->
-  <link name="base">
+<?xml version="1.0" ?>
+<robot name="ur_with_gripper" xmlns:xacro="http://www.ros.org/wiki/xacro" >
+  <!-- UR5e robot arm -->
+  <!-- URDF won't build if following args aren't defined. -->
+  <xacro:arg name="name" default="ur5"/>
+  <xacro:arg name="ur_type" default="ur5"/>
+  <xacro:include filename="$(find ur_description)/urdf/ur.urdf.xacro"/>
+  <!-- end effector -->
+   <link name="rail_gripper_base_link">
     <visual>
       <geometry>
@@ -40,5 +45,5 @@
   <!-- Right finger prismatic joint -->
   <joint name="right_finger_joint" type="prismatic">
-    <parent link="base"/>
+    <parent link="rail_gripper_base_link"/>
     <child link="right_finger"/>
     <origin xyz="0 0.004 0.0" rpy="0 0 0"/>
@@ -48,5 +53,5 @@
   <!-- Left finger prismatic joint (mimics right finger) -->
   <joint name="left_finger_joint" type="prismatic">
-    <parent link="base"/>
+    <parent link="rail_gripper_base_link"/>
     <child link="left_finger"/>
     <origin xyz="0 -0.004 0" rpy="0 0 0"/>
@@ -55,3 +60,7 @@
     <mimic joint="right_finger_joint" multiplier="-1" offset="0"/>
   </joint>
+  <joint name="wrist_3_link_to_gripper_base" type="fixed">
+    <parent link="tool0"/>
+    <child link="rail_gripper_base_link"/>
+  </joint>
 </robot>
