Commit message: End Effector in Rviz on Real Robot

File: src/linear_gripper_visualiser/urdf/linear_gripper.urdf (robot description, URDF)
Before this commit: robot linear_gripper, 3 links, 2 joints
Links:
- removed link base
- added link palm; visual box size=0.0603 0.06 0.06
Joints:
- joint left_finger_joint: parent base -> palm
- joint right_finger_joint: parent base -> palm

File: src/linear_gripper_visualiser/urdf/ur_with_gripper.urdf.xacro (robot description, xacro)
@@ -6,61 +6,9 @@
   <xacro:arg name="ur_type" default="ur5"/>
   <xacro:include filename="$(find ur_description)/urdf/ur.urdf.xacro"/>
-  <!-- end effector -->
-   <link name="rail_gripper_base_link">
-    <visual>
-      <geometry>
-        <box size="0.0603 0.06 0.06"/>
-      </geometry>
-      <origin xyz="0 0 0" rpy="0 0 0"/>
-    </visual>
-  </link>
-  <!-- Right finger -->
-  <link name="right_finger">
-    <visual>
-      <geometry>
-        <box size="0.03625 0.008 0.0335"/>
-      </geometry>
-      <origin xyz="0 0.004 0.0470" rpy="0 0 0"/>
-    </visual>
-    <collision>
-      <geometry>
-        <box size="0.03625 0.008 0.0335"/>
-      </geometry>
-    </collision>
-  </link>
-  <!-- Left finger -->
-  <link name="left_finger">
-    <visual>
-      <geometry>
-        <box size="0.03625 0.008 0.0335"/>
-      </geometry>
-      <origin xyz="0 -0.004 0.0470" rpy="0 0 0"/>
-    </visual>
-    <collision>
-      <geometry>
-        <box size="0.03625 0.008 0.0335"/>
-      </geometry>
-    </collision>
-  </link>
-  <!-- Right finger prismatic joint -->
-  <joint name="right_finger_joint" type="prismatic">
-    <parent link="rail_gripper_base_link"/>
-    <child link="right_finger"/>
-    <origin xyz="0 0.004 0.0" rpy="0 0 0"/>
-    <axis xyz="0 1 0"/>
-    <limit lower="-0.004" upper="0.02" effort="10" velocity="0.05"/>
-  </joint>
-  <!-- Left finger prismatic joint (mimics right finger) -->
-  <joint name="left_finger_joint" type="prismatic">
-    <parent link="rail_gripper_base_link"/>
-    <child link="left_finger"/>
-    <origin xyz="0 -0.004 0" rpy="0 0 0"/>
-    <axis xyz="0 1 0"/>
-    <limit lower="-0.004" upper="0.02" effort="10" velocity="0.05"/>
-    <mimic joint="right_finger_joint" multiplier="-1" offset="0"/>
-  </joint>
-  <joint name="wrist_3_link_to_gripper_base" type="fixed">
+  <xacro:include filename="$(find linear_gripper_visualiser)/urdf/linear_gripper.urdf"/>
+  <joint name="wrist_3_link_to_gripper_palm" type="fixed">
     <parent link="tool0"/>
-    <child link="rail_gripper_base_link"/>
+    <child link="palm"/>
+    <origin xyz="0 0 0.03" rpy="0 0 0"/>
   </joint>
 </robot>

Commit message: Adding movement with URDF

File: src/linear_gripper_visualiser/urdf/linear_gripper.urdf (robot description, URDF)
Before this commit: robot linear_gripper, 3 links, 2 joints
Links:
- link palm: geometry collision box size=0.0603 0.06 0.06; visual box size=0.0603 0.06 0.06

File: src/linear_gripper_visualiser/urdf/ur_with_gripper.urdf.xacro (robot description, xacro)
@@ -10,5 +10,5 @@
     <parent link="tool0"/>
     <child link="palm"/>
-    <origin xyz="0 0 0.03" rpy="0 0 0"/>
+    <origin xyz="0 0 0.04" rpy="0 0 0"/>
   </joint>
 </robot>

Commit message: Final Lab - 3/12/25

File: src/linear_gripper_visualiser/urdf/linear_gripper.urdf (robot description, URDF)
Before this commit: robot linear_gripper, 3 links, 2 joints
Links:
- removed link left_finger
- removed link right_finger
- link palm: geometry visual mesh filename=file://$(find linear_gripper_visualiser)/meshes/gripperURDF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
Joints:
- removed joint left_finger_joint
- removed joint right_finger_joint

File: src/linear_gripper_visualiser/urdf/ur_with_gripper.xacro (robot description, xacro)
@@ -6,9 +6,17 @@
   <xacro:arg name="ur_type" default="ur5"/>
   <xacro:include filename="$(find ur_description)/urdf/ur.urdf.xacro"/>
-  <xacro:include filename="$(find linear_gripper_visualiser)/urdf/linear_gripper.urdf"/>
+  <!-- end effector -->
+  <link name="palm">
+    <visual>
+      <origin xyz="0 0 0" rpy="3.1415 0 0"/>
+      <geometry>
+        <mesh filename="file://$(find linear_gripper_visualiser)/meshes/gripperURDFV2.stl" scale="0.001 0.001 0.001"/>
+      </geometry>
+    </visual>
+  </link>
   <joint name="wrist_3_link_to_gripper_palm" type="fixed">
     <parent link="tool0"/>
     <child link="palm"/>
-    <origin xyz="0 0 0.04" rpy="0 0 0"/>
+    <origin xyz="0 0 0.062" rpy="0 0 0"/>
   </joint>
 </robot>
